Commit message: Can see turtlebot3_burger in rviz - added the .stl mesh files from the turtlebot3 repo - fixed the .urdf.xacro filepaths for the meshes

File: nuturtle_description/urdf/turtlebot3_burger.urdf.xacro (robot description, xacro)
@@ -2,5 +2,5 @@
 <robot name="turtlebot3_burger"
   xmlns:xacro="http://ros.org/wiki/xacro">
-  <!-- <xacro:include filename="$(find turtlebot3_description)/urdf/common_properties.urdf"/> -->
+  <!-- <xacro:include filename="$(find nuturtle_description)/urdf/common_properties.urdf"/> -->
   <!-- Init colour -->
   <material name="black">
@@ -44,5 +44,5 @@
       <origin xyz="-0.032 0 0.0" rpy="0 0 0"/>
       <geometry>
-        <mesh filename="package://turtlebot3_description/meshes/bases/burger_base.stl" scale="0.001 0.001 0.001"/>
+        <mesh filename="package://nuturtle_description/meshes/burger_base.stl" scale="0.001 0.001 0.001"/>
       </geometry>
       <material name="light_black"/>
@@ -70,5 +70,5 @@
       <origin xyz="0 0 0" rpy="1.57 0 0"/>
       <geometry>
-        <mesh filename="package://turtlebot3_description/meshes/wheels/left_tire.stl" scale="0.001 0.001 0.001"/>
+        <mesh filename="package://nuturtle_description/meshes/left_tire.stl" scale="0.001 0.001 0.001"/>
       </geometry>
       <material name="dark"/>
@@ -96,5 +96,5 @@
       <origin xyz="0 0 0" rpy="1.57 0 0"/>
       <geometry>
-        <mesh filename="package://turtlebot3_description/meshes/wheels/right_tire.stl" scale="0.001 0.001 0.001"/>
+        <mesh filename="package://nuturtle_description/meshes/right_tire.stl" scale="0.001 0.001 0.001"/>
       </geometry>
       <material name="dark"/>
@@ -145,5 +145,5 @@
       <origin xyz="0 0 0.0" rpy="0 0 0"/>
       <geometry>
-        <mesh filename="package://turtlebot3_description/meshes/sensors/lds.stl" scale="0.001 0.001 0.001"/>
+        <mesh filename="package://nuturtle_description/meshes/lds.stl" scale="0.001 0.001 0.001"/>
       </geometry>
       <material name="dark"/>

Commit message: Config files being loaded into .urdf.xacro file - made diff_params.yaml file with specified parameters - loading in the parameters and using them - verified that changing the track width changes the wheel distance in rviz

File: nuturtle_description/urdf/turtlebot3_burger.urdf.xacro (robot description, xacro)
@@ -1,6 +1,11 @@
 <?xml version="1.0" ?>
+<!-- This file was taken from the TurtleBot3 repository and modified.-->
 <robot name="turtlebot3_burger"
   xmlns:xacro="http://ros.org/wiki/xacro">
-  <!-- <xacro:include filename="$(find nuturtle_description)/urdf/common_properties.urdf"/> -->
+  <xacro:property name="yaml_file" value="$(find nuturtle_description)/config/diff_params.yaml" />
+  <xacro:property name="props" value="${xacro.load_yaml(yaml_file)['/**']['ros__parameters']}" />
+  <xacro:property name="wheel_radius"  value="${props['wheel_radius']}" />
+  <xacro:property name="track_width"  value="${props['track_width']}" />
+  <xacro:property name="collision_radius"  value="${props['collision_radius']}" />
   <!-- Init colour -->
   <material name="black">
@@ -63,5 +68,5 @@
     <parent link="base_link"/>
     <child link="wheel_left_link"/>
-    <origin xyz="0.0 0.08 0.023" rpy="-1.57 0 0"/>
+    <origin xyz="0.0 ${track_width/2} 0.023" rpy="-1.57 0 0"/>
     <axis xyz="0 0 1"/>
   </joint>
@@ -77,5 +82,5 @@
       <origin xyz="0 0 0" rpy="0 0 0"/>
       <geometry>
-        <cylinder length="0.018" radius="0.033"/>
+        <cylinder length="0.018" radius="${wheel_radius}"/>
       </geometry>
     </collision>
@@ -89,5 +94,5 @@
     <parent link="base_link"/>
     <child link="wheel_right_link"/>
-    <origin xyz="0.0 -0.080 0.023" rpy="-1.57 0 0"/>
+    <origin xyz="0.0 -${track_width/2} 0.023" rpy="-1.57 0 0"/>
     <axis xyz="0 0 1"/>
   </joint>
@@ -103,5 +108,5 @@
       <origin xyz="0 0 0" rpy="0 0 0"/>
       <geometry>
-        <cylinder length="0.018" radius="0.033"/>
+        <cylinder length="0.018" radius="${wheel_radius}"/>
       </geometry>
     </collision>

Commit message: Checking if the collision radius is positive - if it is negative, use the original box geometry. - otherwise, use it as the cylinder radius for collision

File: nuturtle_description/urdf/turtlebot3_burger.urdf.xacro (robot description, xacro)
@@ -56,5 +56,8 @@
       <origin xyz="-0.032 0 0.070" rpy="0 0 0"/>
       <geometry>
-        <box size="0.140 0.140 0.143"/>
+          <cylinder length="0.143" radius="${collision_radius}"/>
+          <xacro:if value = "${collision_radius &lt; 0}">
+            <box size="0.140 0.140 0.143"/>
+          </xacro:if>
       </geometry>
     </collision>

Commit message: Added color functionalities
-added xacro arg for color
-made default color purple, removed the unused colors
-added some choices into the launchfile
-color displaying in rviz correctly

File: nuturtle_description/urdf/turtlebot3_burger.urdf.xacro (robot description, xacro)
@@ -8,13 +8,8 @@
   <xacro:property name="track_width"  value="${props['track_width']}" />
   <xacro:property name="collision_radius"  value="${props['collision_radius']}" />
+  <xacro:arg name="color" default="purple"/>
   <!-- Init colour -->
-  <material name="black">
-      <color rgba="0.0 0.0 0.0 1.0"/>
-  </material>
-  <material name="dark">
-    <color rgba="0.3 0.3 0.3 1.0"/>
-  </material>
-  <material name="light_black">
-    <color rgba="0.4 0.4 0.4 1.0"/>
+  <material name="red">
+    <color rgba="0.8 0.0 0.0 1.0"/>
   </material>
   <material name="blue">
@@ -24,18 +19,9 @@
     <color rgba="0.0 0.8 0.0 1.0"/>
   </material>
-  <material name="grey">
-    <color rgba="0.5 0.5 0.5 1.0"/>
+  <material name="purple">
+    <color rgba="0.3 0.16 0.52 1.0"/>
   </material>
-  <material name="orange">
-    <color rgba="1.0 0.4235 0.0392 1.0"/>
-  </material>
-  <material name="brown">
-    <color rgba="0.8706 0.8118 0.7647 1.0"/>
-  </material>
-  <material name="red">
-    <color rgba="0.8 0.0 0.0 1.0"/>
-  </material>
-  <material name="white">
-    <color rgba="1.0 1.0 1.0 1.0"/>
+  <material name="dark">
+    <color rgba="0.3 0.3 0.3 1.0"/>
   </material>
   <link name="base_footprint"/>
@@ -51,5 +37,5 @@
         <mesh filename="package://nuturtle_description/meshes/burger_base.stl" scale="0.001 0.001 0.001"/>
       </geometry>
-      <material name="light_black"/>
+      <material name="$(arg color)"/>
     </visual>
     <collision>

Commit message: Small fix for the collision geometry logic

File: nuturtle_description/urdf/turtlebot3_burger.urdf.xacro (robot description, xacro)
@@ -42,8 +42,8 @@
       <origin xyz="-0.032 0 0.070" rpy="0 0 0"/>
       <geometry>
-          <cylinder length="0.143" radius="${collision_radius}"/>
           <xacro:if value = "${collision_radius &lt; 0}">
             <box size="0.140 0.140 0.143"/>
           </xacro:if>
+          <cylinder length="0.143" radius="${collision_radius}"/>
       </geometry>
     </collision>
